File: PCB/smd test.kicad_pcb (KiCad board)
At the start: 2 copper layers, 47.5 x 47.5 mm, 136 parts

Commit message: Updated origins, fixed corners, generated initial placement files.
Parts:
- turned REF** to 90 degrees
Other:
- outline, holes or cut-outs redrawn
